Commit message: crontroller works, greedy grasp version

File: ros2_ws/src/aerial_grasping_description/urdf/drone_arm.urdf (robot description, URDF)
Before this commit: robot aerial_robot, 11 links, 10 joints
Links:
- removed link arm_x
- removed link arm_y
- removed link propeller_1
- removed link propeller_2
- removed link propeller_3
- removed link propeller_4
- removed link world
- added link rotor_1_link, mass 0.03; collision cylinder length=0.01 radius=0.07; visual cylinder length=0.01 radius=0.07
- added link rotor_2_link, mass 0.03; collision cylinder length=0.01 radius=0.07; visual cylinder length=0.01 radius=0.07
- added link rotor_3_link, mass 0.03; collision cylinder length=0.01 radius=0.07; visual cylinder length=0.01 radius=0.07
- added link rotor_4_link, mass 0.03; collision cylinder length=0.01 radius=0.07; visual cylinder length=0.01 radius=0.07
- link base_link: geometry collision box size=0.45 0.45 0.08; visual mesh filename=package://aerial_grasping_description/meshes/droneModel_bin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 scale=0.005 0.005 0.005
Joints:
- removed joint base_to_arm_x
- removed joint base_to_arm_y
- removed joint base_to_propeller_1
- removed joint base_to_propeller_2
- removed joint base_to_propeller_3
- removed joint base_to_propeller_4
- removed joint world_to_base
- added joint base_to_rotor_1: type fixed, parent base_link, child rotor_1_link, origin xyz=0.25 0.25 0.05 rpy=0 0 0
- added joint base_to_rotor_2: type fixed, parent base_link, child rotor_2_link, origin xyz=-0.25 0.25 0.05 rpy=0 0 0
- added joint base_to_rotor_3: type fixed, parent base_link, child rotor_3_link, origin xyz=-0.25 -0.25 0.05 rpy=0 0 0
- added joint base_to_rotor_4: type fixed, parent base_link, child rotor_4_link, origin xyz=0.25 -0.25 0.05 rpy=0 0 0
